File: can.kicad_sch (KiCad schematic)
At the start: 16 parts, among them J1 SM04B-GHS, J2 SM04B-GHS, Q1 Q_NMOS_GSD, U2 TJA1051TK/3/1J

Commit message: nearly done with layout
Parts:
- added D17: 1PS79SB30, Diode_SMD:D_SOD-523, symbol Device:D_Schottky
- added F1: Polyfuse, Fuse:Fuse_1206_3216Metric, symbol Device:Polyfuse
- added TP5: VBUS, TestPoint:TestPoint_Pad_1.0x1.0mm, symbol Connector:TestPoint
- J1, J2: symbol Connector_Generic:Conn_01x04 -> Connector_Generic_MountingPin:Conn_01x04_MountingPin
Connections:
- net GND: now also J1.MP (MountPin), J2.MP (MountPin)
- net VIN: now reaches J2.1 (Pin_1)
- net VIN: now also J1.1 (Pin_1), F1.1
- new net: D17.2 (A), F1.2
- new net VBUS: D17.1 (K), TP5.1
- no-connect marks 2 -> 0
Other:
- note added: "VBUS Protection"
