File: passthrough.kicad_sch (KiCad schematic)
At the start: 13 parts, among them J10 MiniFit, J5 Pixhawk 1, J6 Pixhawk 2, J8 DEBUG, Y1 XRCGB16M000FXN20R0

Commit message: nearly done with layout
Parts:
- removed C54, C55: 6p, Capacitor_SMD:C_0402_1005Metric, symbol Device:C
- removed C57: 100n, Capacitor_SMD:C_0402_1005Metric, symbol Device:C
- removed J8: DEBUG, Connector_PinHeader_2.54mm:PinHeader_1x05_P2.54mm_Vertical, symbol Connector_Generic:Conn_01x05
- removed R71: 10K, Resistor_SMD:R_0402_1005Metric, symbol Device:R
- removed R72: 0, Resistor_SMD:R_0402_1005Metric, symbol Device:R
- removed Y1: XRCGB16M000FXN20R0, Crystal:Crystal_SMD_2016-4Pin_2.0x1.6mm, symbol Device:Crystal_GND24
- added C42, C44, C46: 1u, Capacitor_SMD:C_0402_1005Metric, symbol Device:C
- added R47, R69: 10K, Resistor_SMD:R_0402_1005Metric, symbol Device:R
- added R73, R75: R, Resistor_SMD:R_0402_1005Metric, symbol Device:R_Small
- added U17: TA2528, Package_DFN_QFN:WQFN-16-1EP_3x3mm_P0.5mm_EP1.68x1.68mm, symbol Analog_ADC_Extra:TLA2528
- J5, J6: footprint Connector_Molex:Molex_CLIK-Mate_502382-0670_1x06-1MP_P1.25mm_Vertical -> Connector_Molex:Molex_CLIK-Mate_502494-0670_1x06-1MP_P2.00mm_Horizontal; symbol Connector_Generic:Conn_01x06 -> Connector_Generic_MountingPin:Conn_01x06_MountingPin
Connections:
- net +3V3: now also C44.1, C46.1, R47.1, R69.1, U17.10 (DVDD), U17.7 (AVDD)
- net GND: now also J5.MP (MountPin), J6.MP (MountPin), C42.2, C44.2, C46.2, R75.2, U17.17 (GND), U17.9 (GND)
- net SMBUS_SCL renamed SCL
- net SCL: now also R47.2, U17.13 (SCL)
- net SMBUS_SDA renamed SDA
- net SDA: now also R69.2, U17.14 (SDA)
- new net: C42.1, R73.1, U17.8 (DECAP)
- new net: R73.2, R75.1, U17.11 (ADDR)
- new net IESC1: U17.15 (AIN0)
- new net IESC2: U17.16 (AIN1)
- new net IESC3: U17.1 (AIN2)
- new net IESC4: U17.2 (AIN3)
- new net IPAYLOAD: U17.3 (AIN4)
- new net RESV0: U17.4 (AIN5)
- new net RESV1: U17.5 (AIN6)
- new net RESV2: U17.6 (AIN7)
Other:
- note added: "ADDR = 0x10"
- note added: "I2C Pullup"
- note added: "IO Expansion"
- note removed: "16MHz Crystal"
- note removed: "Bridge for testing"
- note removed: "Debug"
- note removed: "Reset Circuitry"
- moved on the sheet: D14, D15, D16, J10
