File: vrb.kicad_sch (KiCad schematic)
At the start: 8 parts, among them J11 XT30, U1 STM32G0B1CBUx

Commit message: nearly done with layout
Parts:
- added J12: Mezzanine, 528850474:CON_528850474_MOL, symbol Connector_Generic:Conn_02x20_Top_Bottom
Connections:
- net CM_PG is gone; now on net CM_STATUS: U1.24 (PB12)
- net +BATT: now also J12.21 (Pin_21), J12.22 (Pin_22), J12.23 (Pin_23), J12.24 (Pin_24), J12.25 (Pin_25), J12.26 (Pin_26), J12.27 (Pin_27), J12.28 (Pin_28), J12.29 (Pin_29), J12.30 (Pin_30), J12.31 (Pin_31), J12.32 (Pin_32)
- net CAN1_STATUS: now also U1.26 (PB14); no longer U1.27 (PB15)
- net CAN1_TERM: now also U1.27 (PB15); no longer U1.26 (PB14)
- net CAN2_SILENT: now also U1.37 (PA15); no longer U1.21 (PB2)
- net CAN2_STATUS: now also U1.44 (PB5); no longer U1.46 (PB7)
- net CAN2_TERM: now also U1.46 (PB7); no longer U1.44 (PB5)
- net CM_EN: now also U1.21 (PB2); no longer U1.32 (PA10/UCPD1_DBCC2)
- net CM_ISENSE: now also U1.22 (PB10); no longer U1.23 (PB11)
- net CM_STATUS: no longer U1.3 (PC15)
- net CM_VSENSE: now also U1.23 (PB11); no longer U1.22 (PB10)
- net FMU1_EN: now also U1.31 (PC7); no longer U1.28 (PA8)
- net FMU1_ISENSE: now also U1.17 (PA6); no longer U1.12 (PA1)
- net FMU1_STATUS: now also U1.32 (PA10/UCPD1_DBCC2); no longer U1.30 (PC6)
- net FMU1_VSENSE: now also U1.18 (PA7); no longer U1.11 (PA0)
- net FMU2_STATUS: now also U1.34 (PA10/PA12); no longer U1.31 (PC7)
- net FMU2_VSENSE: now also U1.11 (PA0); no longer U1.13 (PA2)
- net GND: now also J12.1 (Pin_1), J12.10 (Pin_10), J12.11 (Pin_11), J12.12 (Pin_12), J12.13 (Pin_13), J12.14 (Pin_14), J12.15 (Pin_15), J12.16 (Pin_16), J12.17 (Pin_17), J12.18 (Pin_18), J12.19 (Pin_19), J12.2 (Pin_2), J12.20 (Pin_20), J12.3 (Pin_3), J12.4 (Pin_4), J12.5 (Pin_5), J12.6 (Pin_6), J12.7 (Pin_7), J12.8 (Pin_8), J12.9 (Pin_9)
- net RADAR_EN: now also U1.28 (PA8); no longer U1.34 (PA10/PA12)
- net RADAR_ISENSE: now also U1.16 (PA5); no longer U1.18 (PA7)
- net RADAR_VSENSE: now also U1.15 (PA4); no longer U1.17 (PA6)
- net RADIO_EN: now also U1.30 (PC6); no longer U1.29 (PA9/UCPD1_DBCC1)
- net RADIO_ISENSE: now also U1.13 (PA2); no longer U1.16 (PA5)
- net RADIO_STATUS: now also U1.3 (PC15); no longer U1.1 (PC13)
- net RADIO_VSENSE: now also U1.12 (PA1); no longer U1.15 (PA4)
- net REG_STATUS: now reaches U1.39 (PD1)
- new net IESC1: J12.33 (Pin_33)
- new net IESC2: J12.34 (Pin_34)
- new net IESC3: J12.35 (Pin_35)
- new net IESC4: J12.36 (Pin_36)
- new net IPAYLOAD: J12.37 (Pin_37)
- new net RESV0: J12.38 (Pin_38)
- new net RESV1: J12.39 (Pin_39)
- new net RESV2: J12.40 (Pin_40)
Other:
- added sheet Onboard Regulator (regulator_onboard.kicad_sch)
- added sheet Reset Clock Ctrl (rcc.kicad_sch)
- sheet CANFD 1 (Primary) ports: added VBUS; removed none
- sheet CANFD 2 (Redundant) ports: added VBUS; removed none
- sheet Passthrough Ports ports: added IESC1, IESC2, IESC3, IESC4, IPAYLOAD, RESV0, RESV1, RESV2, SCL, SDA; removed BOOT0, SMBUS_SCL, SMBUS_SDA, SWCLK, SWDIO, UART_TX_DEBUG, XIN, XOUT, nRST
- note added: "Mezzanine PDB Input"
- note added: "TODO: Input power mux?"
- note removed: "TODO: Reset circuitry MCU decoupling 3V3 regulator and power mux Reverse polarity on mini fit Debug connector"
- moved on the sheet: H1, H2, H3, H4, J11
