File: vrb.kicad_sch (KiCad schematic)
At the start: 11 parts, among them J11 XT30, J12 Mezzanine, U1 STM32G0B1CBUx

Commit message: fix capacitor sizes, clean up silkscreen, export
Other:
- sheet Passthrough Ports ports: added RADAR_VOUT; removed none
Changed lines of the file:
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@@
 	(wire
 		(pts
-			(xy 76.2 157.48) (xy 95.25 157.48)
+			(xy 76.2 154.94) (xy 95.25 154.94)
 		)
 		(stroke
@@
 	(wire
 		(pts
-			(xy 76.2 160.02) (xy 95.25 160.02)
+			(xy 76.2 157.48) (xy 95.25 157.48)
 		)
 		(stroke
@@
 	(wire
 		(pts
-			(xy 76.2 154.94) (xy 95.25 154.94)
+			(xy 76.2 152.4) (xy 95.25 152.4)
+		)
+		(stroke
+			(width 0)
+			(type default)
+		)
+	)
+	(wire
+		(pts
+			(xy 76.2 160.02) (xy 95.25 160.02)
 		)
 		(stroke
@@
 	)
 	(label "FMU1_VOUT"
-		(at 76.2 154.94 0)
+		(at 76.2 152.4 0)
 		(effects
 			(font
@@
 	)
 	(label "CM_VOUT"
-		(at 76.2 160.02 0)
+		(at 76.2 157.48 0)
 		(effects
 			(font
@@
 	)
 	(label "FMU2_VOUT"
-		(at 76.2 157.48 0)
+		(at 76.2 154.94 0)
 		(effects
 			(font
@@
 		)
 	)
+	(label "RADAR_VOUT"
+		(at 76.2 160.02 0)
+		(effects
+			(font
+				(size 1.27 1.27)
+			)
+			(justify left bottom)
+		)
+	)
 	(label "RADIO_VOUT"
 		(at 179.07 25.4 0)
@@
 	)
 	(sheet
-		(at 95.25 152.4)
-		(size 19.05 38.1)
+		(at 95.25 149.86)
+		(size 19.05 40.64)
 		(exclude_from_sim no)
 		(in_bom yes)
@@
 		)
 		(property "Sheetname" "Passthrough Ports"
-			(at 95.25 151.6884 0)
+			(at 95.25 149.1484 0)
 			(effects
 				(font
@@
 		)
 		(pin "CM_VOUT" input
-			(at 95.25 160.02 180)
+			(at 95.25 157.48 180)
 			(effects
 				(font
@@
 		)
 		(pin "FMU1_VOUT" input
-			(at 95.25 154.94 180)
+			(at 95.25 152.4 180)
 			(effects
 				(font
@@
 		)
 		(pin "FMU2_VOUT" input
-			(at 95.25 157.48 180)
+			(at 95.25 154.94 180)
 			(effects
 				(font
@@
 			(effects
 				(font
+					(size 1.27 1.27)
+				)
+				(justify left)
+			)
+		)
+		(pin "RADAR_VOUT" input
+			(at 95.25 160.02 180)
+			(effects
+				(font

Commit message: minor revisions
Parts:
- added J14: Conn_01x02, Connector_PinHeader_2.54mm:PinHeader_1x02_P2.54mm_Vertical, symbol Connector_Generic:Conn_01x02
- added R79: 10K, Resistor_SMD:R_0402_1005Metric, symbol Device:R
Connections:
- net +3V3: now also R79.1
- net GND: now also J14.2 (Pin_2)
- net BUTTON: now reaches U1.38 (PD0)
- net BUTTON: now also J14.1 (Pin_1), R79.2
- no-connect marks 3 -> 2
Other:
- note added: "TODO: Make this fault LED powered by VBAT"
