File: vrb.kicad_pcb (KiCad board)
At the start: 2 copper layers, 75 x 69 mm, 174 parts, among them J1 SM04B-GHS, J10 MiniFit, J11 XT30, J2 SM04B-GHS, J3 MiniFit, J4 MiniFit, J5 Pixhawk 1, J6 Pixhawk 2, J7 SM04B-GHS, J8 DEBUG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

Commit message: nearly done with layout
Parts:
- added C40: 100n, Capacitor_SMD:C_0603_1608Metric, F.Cu at (93.3, 129.1)
- added C41: 100n, Capacitor_SMD:C_0603_1608Metric, F.Cu at (96.4, 132.2)
- added C42: 1u, Capacitor_SMD:C_0402_1005Metric, F.Cu at (109.3, 131.7)
- added C43: 1u, Capacitor_SMD:C_0603_1608Metric, F.Cu at (87.5, 127.8)
- added C44: 1u, Capacitor_SMD:C_0402_1005Metric, F.Cu at (111.0, 129.3)
- added C45: 1u, Capacitor_SMD:C_0603_1608Metric, F.Cu at (87.5, 130.3)
- added C46: 1u, Capacitor_SMD:C_0402_1005Metric, F.Cu at (108.2, 131.7)
- added D17: 1PS79SB30, Diode_SMD:D_SOD-523, F.Cu at (86.3, 106.8)
- added D18: GREEN, LED_SMD:LED_0603_1608Metric, F.Cu at (94.4, 126.4)
- added D19: 1PS79SB30, Diode_SMD:D_SOD-523, F.Cu at (86.3, 86.5)
- added F1: Polyfuse, Fuse:Fuse_1206_3216Metric, F.Cu at (82.3, 106.8)
- added F6: Polyfuse, Fuse:Fuse_1206_3216Metric, F.Cu at (82.3, 86.5)
- added J12: Mezzanine, 528850474:CON_528850474_MOL, B.Cu at (109.7, 129.0)
- added R47: 10K, Resistor_SMD:R_0402_1005Metric, F.Cu at (135.8, 123.8)
- added R69: 10K, Resistor_SMD:R_0402_1005Metric, F.Cu at (135.8, 122.8)
- added R70: 1K5, Resistor_SMD:R_0402_1005Metric, F.Cu at (97.2, 126.4)
- added R73: R, Resistor_SMD:R_0402_1005Metric, F.Cu at (111.0, 128.2)
- added R74: 68K, Resistor_SMD:R_0402_1005Metric, F.Cu at (90.9, 128.0)
- added R75: R, Resistor_SMD:R_0402_1005Metric, F.Cu at (111.0, 127.1)
- added R76: 22K, Resistor_SMD:R_0402_1005Metric, F.Cu at (89.8, 128.0)
- added R77: 10K, Resistor_SMD:R_0402_1005Metric, F.Cu at (90.0, 132.7)
- added TP5: VBUS, TestPoint:TestPoint_Pad_1.0x1.0mm, F.Cu at (86.6, 109.1)
- added TP8: VBUS, TestPoint:TestPoint_Pad_1.0x1.0mm, F.Cu at (86.6, 88.8)
- added TP9: 5V, TestPoint:TestPoint_Pad_1.0x1.0mm, F.Cu at (93.6, 131.9)
- added U16: TLV71333PDQN, Package_TO_SOT_SMD:SOT-23-5, F.Cu at (96.4, 129.3)
- added U17: TA2528, Package_DFN_QFN:WQFN-16-1EP_3x3mm_P0.5mm_EP1.68x1.68mm, F.Cu at (107.5, 128.2)
- added U18: TPS2116DRL, Package_TO_SOT_SMD:SOT-583-8, F.Cu at (90.0, 130.6)
- J5, J6: footprint Connector_Molex:Molex_CLIK-Mate_502382-0670_1x06-1MP_P1.25mm_Vertical -> Connector_Molex:Molex_CLIK-Mate_502494-0670_1x06-1MP_P2.00mm_Horizontal
- moved D1 81.6 mm to (80.0, 119.2), turned to -90 degrees
- moved D2 81.5 mm to (80.0, 120.4), turned to -90 degrees
- moved D8 79.9 mm to (80.0, 98.9), turned to -90 degrees
- moved D9 79.9 mm to (80.0, 100.2), turned to -90 degrees
- moved J8 40.4 mm to (126.4, 133.1), turned to 90 degrees
- moved U1 20.2 mm to (128.1, 124.7), turned to -90 degrees
- moved R71 16.0 mm to (123.8, 114.3), turned to -90 degrees
- moved D14 14.9 mm to (136.4, 109.7), turned to 180 degrees
- moved R72 14.8 mm to (124.5, 116.0), turned to 180 degrees
- moved C57 13.6 mm to (125.0, 114.3), turned to 90 degrees
- moved J1 13.6 mm to (76.3, 120.0)
- moved J10 12.7 mm to (140.0, 112.9), turned to -90 degrees
- moved C55 11.0 mm to (126.8, 112.9), turned to 0 degrees
- moved Y1 9.20 mm to (127.2, 115.2), turned to 90 degrees
- moved C38 8.03 mm to (129.0, 118.2), turned to 90 degrees
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Connections:
- J1 pad 1: unconnected-(J1-Pin_1-Pad1) -> /CANFD 2 (Redundant)/VIN
- J1 pad MP: (no net) -> GND
- J2 pad 1: unconnected-(J2-Pin_1-Pad1) -> /CANFD 2 (Redundant)/VIN
- J2 pad MP: (no net) -> GND
- J3 pad 1: /Telemetry Radio/VOUT -> GND
- J3 pad 2: GND -> /Telemetry Radio/VOUT
- J4 pad 1: /RC Radio/VOUT -> GND
- J4 pad 2: GND -> /RC Radio/VOUT
- J5 pad MP: (no net) -> GND
- J6 pad MP: (no net) -> GND
- J7 pad 1: unconnected-(J7-Pin_1-Pad1) -> /CANFD 1 (Primary)/VIN
- J7 pad MP: (no net) -> GND
- J9 pad 1: unconnected-(J9-Pin_1-Pad1) -> /CANFD 1 (Primary)/VIN
- J9 pad MP: (no net) -> GND
- U1 pad 1: /RADIO_STATUS -> unconnected-(U1-PC13-Pad1)
- U1 pad 11: /FMU1_VSENSE -> /FMU2_VSENSE
- U1 pad 12: /FMU1_ISENSE -> /RADIO_VSENSE
- U1 pad 13: /FMU2_VSENSE -> /RADIO_ISENSE
- U1 pad 15: /RADIO_VSENSE -> /RADAR_VSENSE
- U1 pad 16: /RADIO_ISENSE -> /RADAR_ISENSE
- U1 pad 17: /RADAR_VSENSE -> /FMU1_ISENSE
- U1 pad 18: /RADAR_ISENSE -> /FMU1_VSENSE
- U1 pad 21: /CAN2_SILENT -> /CM_EN
- U1 pad 22: /CM_VSENSE -> /CM_ISENSE
- U1 pad 23: /CM_ISENSE -> /CM_VSENSE
- U1 pad 24: /CM_PG -> /CM_STATUS
- U1 pad 26: /CAN1_TERM -> /CAN1_STATUS
- U1 pad 27: /CAN1_STATUS -> /CAN1_TERM
- U1 pad 28: /FMU1_EN -> /RADAR_EN
- U1 pad 29: /RADIO_EN -> unconnected-(U1-PA9/UCPD1_DBCC1-Pad29)
- U1 pad 3: /CM_STATUS -> /RADIO_STATUS
- U1 pad 30: /FMU1_STATUS -> /RADIO_EN
- U1 pad 31: /FMU2_STATUS -> /FMU1_EN
- U1 pad 32: /CM_EN -> /FMU1_STATUS
- U1 pad 34: /RADAR_EN -> /FMU2_STATUS
- U1 pad 37: unconnected-(U1-PA15-Pad37) -> /CAN2_SILENT
- U1 pad 39: unconnected-(U1-PD1-Pad39) -> /REG_STATUS
- U1 pad 44: /CAN2_TERM -> /CAN2_STATUS
- U1 pad 46: /CAN2_STATUS -> /CAN2_TERM
Routing:
- net /FMU1_VSENSE: track 2.43 -> 103.6 mm, vias 1 -> 2
- net /FMU1_ISENSE: track 1.73 -> 89.4 mm
- net /I2C3_SCL_SMBUS: track 0.71 -> 78.3 mm, vias 1 -> 3
- net /FMU1_EN: track 5.49 -> 80.8 mm, vias 1 -> 2
- net /I2C3_SDA_SMBUS: track 1.13 -> 76.1 mm, vias 1 -> 3
- net /CAN2_TERM: track 0.71 -> 74.1 mm, vias 1 -> 2
- net /CAN2_STATUS: track 0.71 -> 73.4 mm, vias 1 -> 2
- net /RADAR_ISENSE: track 1.73 -> 71.4 mm
- net /CAN1_TERM: track 3.38 -> 72.7 mm
- net /FMU1_STATUS: track 1.52 -> 70.7 mm
- net /RADAR_EN: track 5.49 -> 73.5 mm, vias 1 -> 2
- net /RC_STATUS: track 7.19 -> 73.1 mm
- net /CAN1_STATUS: track 1.85 -> 67.3 mm
- net /FMU2_ISENSE: track 1.73 -> 66.0 mm
- net /FDCAN1_TX: track 1.30 -> 64.2 mm
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- added copper zone on In1.Cu, net GND
Other:
- board size 75 x 69 mm -> 75 x 75 mm
- copper layers 2 -> 4
- board text added: "CAN 1"
- board text added: "CAN 2"
- board text added: "FMU 1"
- board text added: "FMU 2"

Commit message: more layout work
Parts:
- moved R75 8.42 mm to (103.9, 131.5), turned to 180 degrees
- moved R73 7.50 mm to (103.9, 130.4), turned to 0 degrees
- moved C44 7.16 mm to (103.9, 129.3), turned to 180 degrees
- moved C42 6.10 mm to (105.6, 126.9), turned to 90 degrees
- moved C46 5.07 mm to (106.7, 126.9), turned to 90 degrees
- moved U17 2.11 mm to (107.3, 130.3), turned to 180 degrees
Routing:
- net /RESV2: track 0.00 -> 13.4 mm, vias 0 -> 1
- net /RESV1: track 0.00 -> 11.3 mm, vias 0 -> 1
- net /RESV0: track 0.00 -> 9.28 mm, vias 0 -> 1
- net /IPAYLOAD: track 0.00 -> 8.71 mm, vias 0 -> 1
- net /IESC4: track 0.00 -> 7.50 mm, vias 0 -> 1
- net /IESC3: track 0.00 -> 6.83 mm, vias 0 -> 1
- net /IESC1: track 0.00 -> 6.34 mm, vias 0 -> 1
- net /IESC2: track 0.00 -> 6.21 mm, vias 0 -> 1
- net /USART1_TX_DEBUG: track 27.1 -> 22.4 mm
- net +3V3: track 17.5 -> 21.7 mm, vias 15 -> 16
- net /CAN2_TERM: track 74.1 -> 70.2 mm
- net /CAN2_STATUS: track 73.4 -> 69.6 mm
- net Net-(U17-ADDR): track 0.00 -> 2.70 mm
- net /CM_ISENSE: track 35.0 -> 37.0 mm
- net Net-(U17-DECAP): track 0.00 -> 1.95 mm
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- added copper zone on B.Cu, net GND
