File: port.kicad_sch (KiCad schematic)
At the start: 16 parts, among them J4 MiniFit, U15 TPS2121

Commit message: nearly done with layout
Connections:
- net GND: now also J4.1 (Pin_1); no longer J4.2 (Pin_2)
- net VOUT: now also J4.2 (Pin_2); no longer J4.1 (Pin_1)
Changed lines of the file:
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@@
 	(symbol
 		(lib_id "Connector_Generic:Conn_01x02")
-		(at 220.98 43.18 0)
+		(at 220.98 45.72 0)
+		(mirror x)
 		(unit 1)
 		(exclude_from_sim no)
@@
 		(on_board yes)
 		(dnp no)
-		(fields_autoplaced yes)
 		(property "Reference" "J4"
-			(at 223.52 43.1799 0)
+			(at 223.52 45.7201 0)
 			(effects
 				(font
@@
 		)
 		(property "Value" "MiniFit"
-			(at 223.52 45.7199 0)
+			(at 223.52 43.1801 0)
 			(effects
 				(font
@@
 		)
 		(property "Footprint" "Connector_Molex:Molex_Mini-Fit_Jr_5569-02A1_2x01_P4.20mm_Horizontal"
-			(at 220.98 43.18 0)
+			(at 220.98 45.72 0)
 			(effects
 				(font
@@
 		)
 		(property "Datasheet" "~"
-			(at 220.98 43.18 0)
+			(at 220.98 45.72 0)
 			(effects
 				(font
@@
 		)
 		(property "Description" "Generic connector, single row, 01x02, script generated (kicad-library-utils/schlib/autogen/connector/)"
-			(at 220.98 43.18 0)
+			(at 220.98 45.72 0)
 			(effects
 				(font

Commit message: fix capacitor sizes, clean up silkscreen, export
Parts:
- J4: footprint Connector_Molex:Molex_Mini-Fit_Jr_5569-02A1_2x01_P4.20mm_Horizontal -> Connector_Molex:Molex_Mini-Fit_Jr_5569-02A2_2x01_P4.20mm_Horizontal
Changed lines of the file:
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@@
 			)
 		)
-		(property "Footprint" "Connector_Molex:Molex_Mini-Fit_Jr_5569-02A1_2x01_P4.20mm_Horizontal"
+		(property "Footprint" "Connector_Molex:Molex_Mini-Fit_Jr_5569-02A2_2x01_P4.20mm_Horizontal"
 			(at 220.98 45.72 0)
 			(effects
